File: kicad/tentacle_v0.5/pcb_octoprobe.kicad_pcb (KiCad board)
At the start: 2 copper layers, 100 x 165 mm, 737 parts, among them J1302 Conn_02x20, J1303 Conn_02x20, J1501 Conn_02x20, J1502 Conn_01x12, J201 Conn_02x05, J202 Conn_01x5, J301 USB_C_Receptacle_USB2.0, J501 Conn_02x20, U1001 GAQY221S, U1101 GAQY221S, U1201 GAQY221S, U1501 RP2040, U1502 W25Q32JVS, U1503 TXB0108PW, U201 RP2040, U202 AMS1117-3.3, U203 W25Q32JVS, U204 TPS2595xx, U205 TPS2595xx, U207 TPS2595xx, U302 USB2514B_Bi, U601 GAQY221S, U701 GAQY221S, U801 GAQY221S, U901 GAQY221S, X201 Oscillator-12MHz, Y301 24MHz

Commit message: Ordered tentacle v0.5 at jlcpcb
Parts:
- added ?: prototype_NC, 00_project_library:octoprobe_breakout_PB_NC, F.Cu at (127.4, 96.0)
- added ?: prototype_NC, 00_project_library:octoprobe_breakout_PB_NC, F.Cu at (96.9, 101.1)
- added ?: prototype_NC, 00_project_library:octoprobe_breakout_PB_NC, F.Cu at (94.4, 157.0)
- added ?: prototype_NC, 00_project_library:octoprobe_breakout_PB_NC, F.Cu at (91.8, 172.2)
- added ?: prototype_NC, 00_project_library:octoprobe_breakout_PB_NC, F.Cu at (101.9, 98.6)
- added ?: prototype_NC, 00_project_library:octoprobe_breakout_PB_NC, F.Cu at (99.4, 93.5)
- added ?: prototype_NC, 00_project_library:octoprobe_breakout_PB_NC, F.Cu at (114.6, 101.1)
- added ?: prototype_NC, 00_project_library:octoprobe_breakout_PB_NC, F.Cu at (129.9, 157.0)
- added ?: prototype_NC, 00_project_library:octoprobe_breakout_PB_NC, F.Cu at (109.5, 169.7)
- added ?: prototype_NC, 00_project_library:octoprobe_breakout_PB_NC, F.Cu at (61.3, 141.7)
- added ?: prototype_NC, 00_project_library:octoprobe_breakout_PB_NC, F.Cu at (127.3, 162.1)
- added ?: prototype_NC, 00_project_library:octoprobe_breakout_PB_NC, F.Cu at (124.8, 93.5)
- added ?: prototype_NC, 00_project_library:octoprobe_breakout_PB_NC, F.Cu at (61.3, 118.9)
- added ?: prototype_NC, 00_project_library:octoprobe_breakout_PB_NC, F.Cu at (94.3, 162.1)
- added ?: prototype_NC, 00_project_library:octoprobe_breakout_PB_NC, F.Cu at (117.2, 98.6)
- added ?: prototype_NC, 00_project_library:octoprobe_breakout_PB_NC, F.Cu at (61.3, 129.0)
- added ?: prototype_NC, 00_project_library:octoprobe_breakout_PB_NC, F.Cu at (61.3, 134.1)
- added ?: prototype_NC, 00_project_library:octoprobe_breakout_PB_NC, F.Cu at (107.1, 96.0)
- added ?: prototype_NC, 00_project_library:octoprobe_breakout_PB_NC, F.Cu at (101.9, 169.7)
- added ?: prototype_NC, 00_project_library:octoprobe_breakout_PB_NC, F.Cu at (109.6, 154.4)
- added ?: prototype_NC, 00_project_library:octoprobe_breakout_PB_NC, F.Cu at (129.9, 96.0)
- added ?: prototype_NC, 00_project_library:octoprobe_breakout_PB_NC, F.Cu at (96.9, 154.4)
- added ?: prototype_NC, 00_project_library:octoprobe_breakout_PB_NC, F.Cu at (61.3, 111.3)
- added ?: prototype_NC, 00_project_library:octoprobe_breakout_PB_NC, F.Cu at (104.5, 159.5)
- added ?: prototype_NC, 00_project_library:octoprobe_breakout_PB_NC, F.Cu at (114.6, 167.1)
- added ?: prototype_NC, 00_project_library:octoprobe_breakout_PB_NC, F.Cu at (109.6, 167.1)
- added ?: prototype_NC, 00_project_library:octoprobe_breakout_PB_NC, F.Cu at (119.7, 172.2)
- added ?: prototype_NC, 00_project_library:octoprobe_breakout_PB_NC, F.Cu at (91.8, 164.6)
- added ?: prototype_NC, 00_project_library:octoprobe_breakout_PB_NC, F.Cu at (61.3, 124.0)
- added ?: prototype_NC, 00_project_library:octoprobe_breakout_PB_NC, F.Cu at (109.6, 162.1)
- added ?: prototype_NC, 00_project_library:octoprobe_breakout_PB_NC, F.Cu at (109.6, 157.0)
- added ?: prototype_NC, 00_project_library:octoprobe_breakout_PB_NC, F.Cu at (91.9, 96.0)
- added ?: prototype_NC, 00_project_library:octoprobe_breakout_PB_NC, F.Cu at (61.3, 151.9)
- added ?: prototype_NC, 00_project_library:octoprobe_breakout_PB_NC, F.Cu at (61.3, 139.2)
- added ?: prototype_NC, 00_project_library:octoprobe_breakout_PB_NC, F.Cu at (117.2, 96.0)
- added ?: prototype_NC, 00_project_library:octoprobe_breakout_PB_NC, F.Cu at (96.9, 93.5)
- added ?: prototype_NC, 00_project_library:octoprobe_breakout_PB_NC, F.Cu at (102.0, 154.4)
- added ?: prototype_NC, 00_project_library:octoprobe_breakout_PB_NC, F.Cu at (94.3, 164.6)
- added ?: prototype_NC, 00_project_library:octoprobe_breakout_PB_NC, F.Cu at (117.2, 167.1)
- added ?: prototype_NC, 00_project_library:octoprobe_breakout_PB_NC, F.Cu at (127.4, 157.0)
- added ?: prototype_NC, 00_project_library:octoprobe_breakout_PB_NC, F.Cu at (122.3, 167.1)
- added ?: prototype_NC, 00_project_library:octoprobe_breakout_PB_NC, F.Cu at (99.4, 162.1)
- added ?: prototype_NC, 00_project_library:octoprobe_breakout_PB_NC, F.Cu at (99.4, 159.5)
- added ?: prototype_NC, 00_project_library:octoprobe_breakout_PB_NC, F.Cu at (112.1, 167.1)
- added ?: prototype_NC, 00_project_library:octoprobe_breakout_PB_NC, F.Cu at (124.8, 159.5)
- added ?: prototype_NC, 00_project_library:octoprobe_breakout_PB_NC, F.Cu at (127.4, 154.4)
- added ?: prototype_NC, 00_project_library:octoprobe_breakout_PB_NC, F.Cu at (112.1, 169.7)
- added ?: prototype_NC, 00_project_library:octoprobe_breakout_PB_NC, F.Cu at (99.4, 96.0)
- added ?: prototype_NC, 00_project_library:octoprobe_breakout_PB_NC, F.Cu at (61.3, 131.6)
- added ?: prototype_NC, 00_project_library:octoprobe_breakout_PB_NC, F.Cu at (99.4, 164.6)
- added ?: prototype_NC, 00_project_library:octoprobe_breakout_PB_NC, F.Cu at (114.7, 157.0)
- added ?: prototype_NC, 00_project_library:octoprobe_breakout_PB_NC, F.Cu at (117.2, 157.0)
- added ?: prototype_NC, 00_project_library:octoprobe_breakout_PB_NC, F.Cu at (61.3, 126.5)
- added ?: prototype_NC, 00_project_library:octoprobe_breakout_PB_NC, F.Cu at (104.5, 162.1)
- added ?: prototype_NC, 00_project_library:octoprobe_breakout_PB_NC, F.Cu at (112.1, 101.1)
- added ?: prototype_NC, 00_project_library:octoprobe_breakout_PB_NC, F.Cu at (124.8, 172.2)
- added ?: prototype_NC, 00_project_library:octoprobe_breakout_PB_NC, F.Cu at (124.8, 157.0)
- added ?: prototype_NC, 00_project_library:octoprobe_breakout_PB_NC, F.Cu at (104.4, 169.7)
- added ?: prototype_NC, 00_project_library:octoprobe_breakout_PB_NC, F.Cu at (117.2, 164.6)
- added ?: prototype_NC, 00_project_library:octoprobe_breakout_PB_NC, F.Cu at (91.9, 93.5)
- added ?: prototype_NC, 00_project_library:octoprobe_breakout_PB_NC, F.Cu at (104.5, 96.0)
- added ?: prototype_NC, 00_project_library:octoprobe_breakout_PB_NC, F.Cu at (109.6, 93.5)
- added ?: prototype_NC, 00_project_library:octoprobe_breakout_PB_NC, F.Cu at (94.4, 96.0)
- added ?: prototype_NC, 00_project_library:octoprobe_breakout_PB_NC, F.Cu at (119.7, 98.6)
- added ?: prototype_NC, 00_project_library:octoprobe_breakout_PB_NC, F.Cu at (129.8, 169.7)
- added ?: prototype_NC, 00_project_library:octoprobe_breakout_PB_NC, F.Cu at (129.9, 154.4)
- added ?: prototype_NC, 00_project_library:octoprobe_breakout_PB_NC, F.Cu at (96.8, 172.2)
- added ?: prototype_NC, 00_project_library:octoprobe_breakout_PB_NC, F.Cu at (112.1, 164.6)
- added ?: prototype_NC, 00_project_library:octoprobe_breakout_PB_NC, F.Cu at (107.1, 154.4)
- added ?: prototype_NC, 00_project_library:octoprobe_breakout_PB_NC, F.Cu at (127.3, 172.2)
- added ?: prototype_NC, 00_project_library:octoprobe_breakout_PB_NC, F.Cu at (104.5, 157.0)
- added ?: prototype_NC, 00_project_library:octoprobe_breakout_PB_NC, F.Cu at (96.9, 167.1)
- added ?: prototype_NC, 00_project_library:octoprobe_breakout_PB_NC, F.Cu at (107.0, 159.5)
- added ?: prototype_NC, 00_project_library:octoprobe_breakout_PB_NC, F.Cu at (99.4, 167.1)
- added ?: prototype_NC, 00_project_library:octoprobe_breakout_PB_NC, F.Cu at (109.6, 101.1)
- added ?: prototype_NC, 00_project_library:octoprobe_breakout_PB_NC, F.Cu at (96.9, 98.6)
- added ?: prototype_NC, 00_project_library:octoprobe_breakout_PB_NC, F.Cu at (117.2, 154.4)
- added ?: prototype_NC, 00_project_library:octoprobe_breakout_PB_NC, F.Cu at (119.8, 157.0)
- added ?: prototype_NC, 00_project_library:octoprobe_breakout_PB_NC, F.Cu at (112.1, 98.6)
- added ?: prototype_NC, 00_project_library:octoprobe_breakout_PB_NC, F.Cu at (124.8, 101.1)
- added ?: prototype_NC, 00_project_library:octoprobe_breakout_PB_NC, F.Cu at (114.6, 98.6)
- added ?: prototype_NC, 00_project_library:octoprobe_breakout_PB_NC, F.Cu at (61.3, 116.3)
- added ?: prototype_NC, 00_project_library:octoprobe_breakout_PB_NC, F.Cu at (96.9, 164.6)
- added ?: prototype_NC, 00_project_library:octoprobe_breakout_PB_NC, F.Cu at (112.1, 93.5)
- added ?: prototype_NC, 00_project_library:octoprobe_breakout_PB_NC, F.Cu at (114.6, 172.2)
- added ?: prototype_NC, 00_project_library:octoprobe_breakout_PB_NC, F.Cu at (102.0, 93.5)
- added ?: prototype_NC, 00_project_library:octoprobe_breakout_PB_NC, F.Cu at (127.3, 164.6)
- added ?: prototype_NC, 00_project_library:octoprobe_breakout_PB_NC, F.Cu at (124.8, 167.1)
- added ?: prototype_NC, 00_project_library:octoprobe_breakout_PB_NC, F.Cu at (112.1, 172.2)
- added ?: prototype_NC, 00_project_library:octoprobe_breakout_PB_NC, F.Cu at (61.3, 121.4)
- added ?: prototype_NC, 00_project_library:octoprobe_breakout_PB_NC, F.Cu at (122.3, 93.5)
- added ?: prototype_NC, 00_project_library:octoprobe_breakout_PB_NC, F.Cu at (101.9, 172.2)
- added ?: prototype_NC, 00_project_library:octoprobe_breakout_PB_NC, F.Cu at (109.6, 98.6)
- added ?: prototype_NC, 00_project_library:octoprobe_breakout_PB_NC, F.Cu at (91.8, 167.2)
- added ?: prototype_NC, 00_project_library:octoprobe_breakout_PB_NC, F.Cu at (94.3, 98.6)
- added ?: prototype_NC, 00_project_library:octoprobe_breakout_PB_NC, F.Cu at (99.4, 157.0)
- added ?: prototype_NC, 00_project_library:octoprobe_breakout_PB_NC, F.Cu at (104.5, 98.6)
- added ?: prototype_NC, 00_project_library:octoprobe_breakout_PB_NC, F.Cu at (122.3, 159.5)
- added ?: prototype_NC, 00_project_library:octoprobe_breakout_PB_NC, F.Cu at (109.6, 159.5)
- added ?: prototype_NC, 00_project_library:octoprobe_breakout_PB_NC, F.Cu at (107.0, 172.2)
- added ?: prototype_NC, 00_project_library:octoprobe_breakout_PB_NC, F.Cu at (122.3, 162.1)
- added ?: prototype_NC, 00_project_library:octoprobe_breakout_PB_NC, F.Cu at (94.4, 154.4)
- added ?: prototype_NC, 00_project_library:octoprobe_breakout_PB_NC, F.Cu at (104.5, 164.6)
- added ?: prototype_NC, 00_project_library:octoprobe_breakout_PB_NC, F.Cu at (127.3, 101.1)
- added ?: prototype_NC, 00_project_library:octoprobe_breakout_PB_NC, F.Cu at (94.3, 169.7)
- added ?: prototype_NC, 00_project_library:octoprobe_breakout_PB_NC, F.Cu at (127.3, 98.6)
- added ?: prototype_NC, 00_project_library:octoprobe_breakout_PB_NC, F.Cu at (129.9, 159.5)
- added ?: prototype_NC, 00_project_library:octoprobe_breakout_PB_NC, F.Cu at (91.8, 98.6)
- added ?: prototype_NC, 00_project_library:octoprobe_breakout_PB_NC, F.Cu at (124.8, 96.0)
- added ?: prototype_NC, 00_project_library:octoprobe_breakout_PB_NC, F.Cu at (104.4, 172.2)
- added ?: prototype_NC, 00_project_library:octoprobe_breakout_PB_NC, F.Cu at (129.9, 164.6)
- added ?: prototype_NC, 00_project_library:octoprobe_breakout_PB_NC, F.Cu at (122.3, 154.4)
- added ?: prototype_NC, 00_project_library:octoprobe_breakout_PB_NC, F.Cu at (107.0, 169.7)
- added ?: prototype_NC, 00_project_library:octoprobe_breakout_PB_NC, F.Cu at (119.7, 169.7)
- added ?: prototype_NC, 00_project_library:octoprobe_breakout_PB_NC, F.Cu at (94.3, 101.1)
- added ?: prototype_NC, 00_project_library:octoprobe_breakout_PB_NC, F.Cu at (61.3, 144.3)
- added ?: prototype_NC, 00_project_library:octoprobe_breakout_PB_NC, F.Cu at (104.5, 167.1)
- added ?: prototype_NC, 00_project_library:octoprobe_breakout_PB_NC, F.Cu at (114.6, 162.1)
- added ?: prototype_NC, 00_project_library:octoprobe_breakout_PB_NC, F.Cu at (124.8, 169.7)
- added ?: prototype_NC, 00_project_library:octoprobe_breakout_PB_NC, F.Cu at (101.9, 159.5)
- added ?: prototype_NC, 00_project_library:octoprobe_breakout_PB_NC, F.Cu at (104.5, 101.1)
- added ?: prototype_NC, 00_project_library:octoprobe_breakout_PB_NC, F.Cu at (99.4, 169.7)
- added ?: prototype_NC, 00_project_library:octoprobe_breakout_PB_NC, F.Cu at (104.5, 154.4)
- added ?: prototype_NC, 00_project_library:octoprobe_breakout_PB_NC, F.Cu at (117.1, 172.2)
- added ?: prototype_NC, 00_project_library:octoprobe_breakout_PB_NC, F.Cu at (122.3, 96.0)
- added ?: prototype_NC, 00_project_library:octoprobe_breakout_PB_NC, F.Cu at (61.3, 149.4)
- added ?: prototype_NC, 00_project_library:octoprobe_breakout_PB_NC, F.Cu at (107.0, 164.6)
- added ?: prototype_NC, 00_project_library:octoprobe_breakout_PB_NC, F.Cu at (101.9, 167.1)
- added ?: prototype_NC, 00_project_library:octoprobe_breakout_PB_NC, F.Cu at (114.7, 96.0)
- added ?: prototype_NC, 00_project_library:octoprobe_breakout_PB_NC, F.Cu at (101.9, 164.6)
- added ?: prototype_NC, 00_project_library:octoprobe_breakout_PB_NC, F.Cu at (107.0, 167.1)
- added ?: prototype_NC, 00_project_library:octoprobe_breakout_PB_NC, F.Cu at (91.9, 157.0)
- added ?: prototype_NC, 00_project_library:octoprobe_breakout_PB_NC, F.Cu at (122.2, 172.2)
- added ?: prototype_NC, 00_project_library:octoprobe_breakout_PB_NC, F.Cu at (102.0, 157.0)
- added ?: prototype_NC, 00_project_library:octoprobe_breakout_PB_NC, F.Cu at (119.7, 164.6)
- added ?: prototype_NC, 00_project_library:octoprobe_breakout_PB_NC, F.Cu at (61.3, 136.7)
- added ?: prototype_NC, 00_project_library:octoprobe_breakout_PB_NC, F.Cu at (104.5, 93.5)
- added ?: prototype_NC, 00_project_library:octoprobe_breakout_PB_NC, F.Cu at (61.3, 106.2)
- added ?: prototype_NC, 00_project_library:octoprobe_breakout_PB_NC, F.Cu at (127.3, 159.5)
- added ?: prototype_NC, 00_project_library:octoprobe_breakout_PB_NC, F.Cu at (119.7, 162.1)
- added ?: prototype_NC, 00_project_library:octoprobe_breakout_PB_NC, F.Cu at (127.4, 93.5)
- added ?: prototype_NC, 00_project_library:octoprobe_breakout_PB_NC, F.Cu at (99.4, 172.2)
- added ?: prototype_NC, 00_project_library:octoprobe_breakout_PB_NC, F.Cu at (94.3, 172.2)
- added ?: prototype_NC, 00_project_library:octoprobe_breakout_PB_NC, F.Cu at (61.3, 108.7)
- added ?: prototype_NC, 00_project_library:octoprobe_breakout_PB_NC, F.Cu at (117.1, 169.7)
- added ?: prototype_NC, 00_project_library:octoprobe_breakout_PB_NC, F.Cu at (61.3, 146.8)
- added ?: prototype_NC, 00_project_library:octoprobe_breakout_PB_NC, F.Cu at (127.3, 167.1)
- added ?: prototype_NC, 00_project_library:octoprobe_breakout_PB_NC, F.Cu at (117.2, 162.1)
- added ?: prototype_NC, 00_project_library:octoprobe_breakout_PB_NC, F.Cu at (114.6, 159.5)
- added ?: prototype_NC, 00_project_library:octoprobe_breakout_PB_NC, F.Cu at (119.7, 159.5)
- added ?: prototype_NC, 00_project_library:octoprobe_breakout_PB_NC, F.Cu at (124.8, 162.1)
- added ?: prototype_NC, 00_project_library:octoprobe_breakout_PB_NC, F.Cu at (112.1, 159.5)
- added ?: prototype_NC, 00_project_library:octoprobe_breakout_PB_NC, F.Cu at (99.4, 98.6)
- added ?: prototype_NC, 00_project_library:octoprobe_breakout_PB_NC, F.Cu at (129.9, 167.1)
- added ?: prototype_NC, 00_project_library:octoprobe_breakout_PB_NC, F.Cu at (129.8, 172.2)
- added ?: prototype_NC, 00_project_library:octoprobe_breakout_PB_NC, F.Cu at (107.0, 98.6)
- added ?: prototype_NC, 00_project_library:octoprobe_breakout_PB_NC, F.Cu at (96.9, 162.1)
- added ?: prototype_NC, 00_project_library:octoprobe_breakout_PB_NC, F.Cu at (129.9, 98.6)
- added ?: prototype_NC, 00_project_library:octoprobe_breakout_PB_NC, F.Cu at (124.8, 98.6)
- added ?: prototype_NC, 00_project_library:octoprobe_breakout_PB_NC, F.Cu at (107.0, 101.1)
- added ?: prototype_NC, 00_project_library:octoprobe_breakout_PB_NC, F.Cu at (107.1, 157.0)
- added ?: prototype_NC, 00_project_library:octoprobe_breakout_PB_NC, F.Cu at (122.3, 157.0)
- added ?: prototype_NC, 00_project_library:octoprobe_breakout_PB_NC, F.Cu at (101.9, 162.1)
- added ?: prototype_NC, 00_project_library:octoprobe_breakout_PB_NC, F.Cu at (119.7, 101.1)
- added ?: prototype_NC, 00_project_library:octoprobe_breakout_PB_NC, F.Cu at (107.0, 162.1)
- added ?: prototype_NC, 00_project_library:octoprobe_breakout_PB_NC, F.Cu at (94.3, 167.1)
- added ?: prototype_NC, 00_project_library:octoprobe_breakout_PB_NC, F.Cu at (119.7, 167.1)
- added ?: prototype_NC, 00_project_library:octoprobe_breakout_PB_NC, F.Cu at (129.9, 162.1)
- added ?: prototype_NC, 00_project_library:octoprobe_breakout_PB_NC, F.Cu at (122.3, 164.6)
- added ?: prototype_NC, 00_project_library:octoprobe_breakout_PB_NC, F.Cu at (119.8, 96.0)
- added ?: prototype_NC, 00_project_library:octoprobe_breakout_PB_NC, F.Cu at (122.3, 98.6)
- added ?: prototype_NC, 00_project_library:octoprobe_breakout_PB_NC, F.Cu at (91.8, 159.5)
- added ?: prototype_NC, 00_project_library:octoprobe_breakout_PB_NC, F.Cu at (119.8, 154.4)
- added ?: prototype_NC, 00_project_library:octoprobe_breakout_PB_NC, F.Cu at (114.7, 93.5)
- added ?: prototype_NC, 00_project_library:octoprobe_breakout_PB_NC, F.Cu at (109.6, 164.6)
- added ?: prototype_NC, 00_project_library:octoprobe_breakout_PB_NC, F.Cu at (112.1, 96.0)
- added ?: prototype_NC, 00_project_library:octoprobe_breakout_PB_NC, F.Cu at (114.6, 169.7)
- added ?: prototype_NC, 00_project_library:octoprobe_breakout_PB_NC, F.Cu at (61.3, 113.8)
- added ?: prototype_NC, 00_project_library:octoprobe_breakout_PB_NC, F.Cu at (129.9, 101.1)
- added ?: prototype_NC, 00_project_library:octoprobe_breakout_PB_NC, F.Cu at (91.8, 101.1)
- added ?: prototype_NC, 00_project_library:octoprobe_breakout_PB_NC, F.Cu at (96.9, 96.0)
- added ?: prototype_NC, 00_project_library:octoprobe_breakout_PB_NC, F.Cu at (122.2, 169.7)
- added ?: prototype_NC, 00_project_library:octoprobe_breakout_PB_NC, F.Cu at (94.3, 159.5)
- added ?: prototype_NC, 00_project_library:octoprobe_breakout_PB_NC, F.Cu at (96.9, 159.5)
- added ?: prototype_NC, 00_project_library:octoprobe_breakout_PB_NC, F.Cu at (117.2, 101.1)
- added ?: prototype_NC, 00_project_library:octoprobe_breakout_PB_NC, F.Cu at (109.5, 172.2)
- added ?: prototype_NC, 00_project_library:octoprobe_breakout_PB_NC, F.Cu at (112.1, 162.1)
- added ?: prototype_NC, 00_project_library:octoprobe_breakout_PB_NC, F.Cu at (124.8, 154.4)
- added ?: prototype_NC, 00_project_library:octoprobe_breakout_PB_NC, F.Cu at (114.7, 154.4)
- added ?: prototype_NC, 00_project_library:octoprobe_breakout_PB_NC, F.Cu at (107.1, 93.5)
- added ?: prototype_NC, 00_project_library:octoprobe_breakout_PB_NC, F.Cu at (99.4, 154.4)
- added ?: prototype_NC, 00_project_library:octoprobe_breakout_PB_NC, F.Cu at (117.2, 93.5)
- added ?: prototype_NC, 00_project_library:octoprobe_breakout_PB_NC, F.Cu at (61.3, 103.6)
- added ?: prototype_NC, 00_project_library:octoprobe_breakout_PB_NC, F.Cu at (122.3, 101.1)
- added ?: prototype_NC, 00_project_library:octoprobe_breakout_PB_NC, F.Cu at (96.9, 157.0)
- added ?: prototype_NC, 00_project_library:octoprobe_breakout_PB_NC, F.Cu at (109.6, 96.0)
- added ?: prototype_NC, 00_project_library:octoprobe_breakout_PB_NC, F.Cu at (119.8, 93.5)
- added ?: prototype_NC, 00_project_library:octoprobe_breakout_PB_NC, F.Cu at (129.9, 93.5)
- added ?: prototype_NC, 00_project_library:octoprobe_breakout_PB_NC, F.Cu at (112.1, 154.4)
- added ?: prototype_NC, 00_project_library:octoprobe_breakout_PB_NC, F.Cu at (94.4, 93.5)
- added ?: prototype_NC, 00_project_library:octoprobe_breakout_PB_NC, F.Cu at (101.9, 101.1)
- added ?: prototype_NC, 00_project_library:octoprobe_breakout_PB_NC, F.Cu at (127.3, 169.7)
- added ?: prototype_NC, 00_project_library:octoprobe_breakout_PB_NC, F.Cu at (91.9, 154.4)
- added ?: prototype_NC, 00_project_library:octoprobe_breakout_PB_NC, F.Cu at (117.2, 159.5)
- added ?: prototype_NC, 00_project_library:octoprobe_breakout_PB_NC, F.Cu at (99.4, 101.1)
- added ?: prototype_NC, 00_project_library:octoprobe_breakout_PB_NC, F.Cu at (91.8, 169.7)
- added ?: prototype_NC, 00_project_library:octoprobe_breakout_PB_NC, F.Cu at (124.8, 164.6)
- added ?: prototype_NC, 00_project_library:octoprobe_breakout_PB_NC, F.Cu at (112.1, 157.0)
- added ?: prototype_NC, 00_project_library:octoprobe_breakout_PB_NC, F.Cu at (91.8, 162.1)
- added ?: prototype_NC, 00_project_library:octoprobe_breakout_PB_NC, F.Cu at (96.8, 169.7)
- added ?: prototype_NC, 00_project_library:octoprobe_breakout_PB_NC, F.Cu at (114.6, 164.6)
- added ?: prototype_NC, 00_project_library:octoprobe_breakout_PB_NC, F.Cu at (102.0, 96.0)
- C216: value 470u -> 1000u; footprint Capacitor_SMD:C_Elec_6.3x5.8 -> Capacitor_THT:CP_Radial_D8.0mm_P2.50mm
- R103, R104, R301: value 2k2 -> 4K7
- R201, R204: value 1k -> 1K
- X201: footprint Oscillator:Oscillator_SMD_ECS_2520MV-xxx-xx-4Pin_2.5x2.0mm -> Crystal:Crystal_SMD_2520-4Pin_2.5x2.0mm
- moved TH1302 7.65 mm to (147.0, 171.3)
- moved C202 4.38 mm to (85.4, 29.6)
- moved U202 4.38 mm to (91.5, 29.6)
- moved C216 3.29 mm to (99.2, 25.3)
- moved X201 0.58 mm to (121.1, 47.9)
- moved C1507 0.06 mm to (124.1, 45.6)
Connections:
- net Net-(U201-GPIO20) renamed /RP2 CPU/LED_ERR
- net Net-(U201-GPIO24) renamed /RP2 CPU/LED_ACTIVE
Routing:
- net +3V3infra: track 420.5 -> 414.3 mm
- net +5Vbuf: track 88.4 -> 87.1 mm
- net RELAIS_6: track 13.5 -> 12.9 mm
- net GND: track 159.5 -> 159.3 mm, vias 133 -> 400
Other:
- board text added: "Octoprobe tentacle"
- board text added: "serial"
- board text removed: "Octo"
- board text removed: "probe"
- board text removed: "tentacle"
