File: kicad/tentacle_v0.5/pcb_octoprobe_relay_breakout.kicad_sch (KiCad schematic)
At the start: 1 part, among them J501 Conn_02x20

Commit message: Breadboard: Remove pads from schematic
Connections:
- net +3V3 renamed +3V3infra
Changed lines of the file:
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@@
 	)
 	(symbol
-		(lib_id "power:+3V3")
+		(lib_id "00_project_library:+3V3infra")
 		(at 179.07 43.18 0)
 		(unit 1)
@@
 			)
 		)
-		(property "Value" "+3V3"
+		(property "Value" "+3V3infra"
 			(at 179.0701 39.37 90)
 			(effects
