File: kicad/tentacle_v0.6/pcb_octoprobe.kicad_sch (KiCad schematic)
At the start: 10 parts, among them J202 Conn_01x5

Commit message: Tentacle v0.6
Connections:
- net +3V3dut renamed +5Vdut
Changed lines of the file:
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@@
 	)
 	(symbol
-		(lib_id "00_project_library:+3V3dut")
+		(lib_id "00_project_library:+5Vdut")
 		(at 125.73 100.33 0)
 		(unit 1)
@@
 			)
 		)
-		(property "Value" "+3V3dut"
+		(property "Value" "+5Vdut"
 			(at 125.73 96.266 90)
 			(effects
