File: kicad/tentacle_v0.6/pcb_octoprobe_cpu.kicad_sch (KiCad schematic)
At the start: 27 parts, among them J201 Conn_02x05, U201 RP2040, U203 W25Q32JVS, X201 Oscillator-12MHz

Commit message: Tentacle v0.6: hw_version 0x01->0x02
Connections:
- net HW_VERSION_0: now reaches U201.37 (GPIO25)
- net HW_VERSION_0: now also R210.1, U201.39 (GPIO27/ADC1), U201.40 (GPIO28/ADC2), U201.41 (GPIO29/ADC3); no longer R213.1
- new net HW_VERSION_1: R213.1, U201.38 (GPIO26/ADC0)
Other:
- note added: "HW version: 0x02"
- note removed: "HW version: 0x01"
- moved on the sheet: R210, R213

Commit message: Tentacle v0.6
Parts:
- R202, R203: value 27R -> 33R
Connections:
- net HW_VERSION_0: no longer names the net of R210.1, U201.37 (GPIO25), U201.39 (GPIO27/ADC1), U201.40 (GPIO28/ADC2), U201.41 (GPIO29/ADC3)
- net HW_VERSION_1: no longer names the net of R213.1, U201.38 (GPIO26/ADC0)
Other:
- note added: "0x01 hw_version"
- note added: "0x02 hw_version"
- note added: "0x04 hw_version"
- note added: "0x08 hw_version"
- note added: "0x16 hw_version"
Changed lines of the file:
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@@
 		)
 	)
+	(text "0x08 hw_version"
+		(exclude_from_sim no)
+		(at 134.62 96.266 0)
+		(effects
+			(font
+				(size 1.27 1.27)
+			)
+			(justify left bottom)
+		)
+	)
+	(text "0x01 hw_version"
+		(exclude_from_sim no)
+		(at 135.128 104.14 0)
+		(effects
+			(font
+				(size 1.27 1.27)
+			)
+			(justify left bottom)
+		)
+	)
+	(text "0x16 hw_version"
+		(exclude_from_sim no)
+		(at 134.62 93.726 0)
+		(effects
+			(font
+				(size 1.27 1.27)
+			)
+			(justify left bottom)
+		)
+	)
+	(text "0x04 hw_version"
+		(exclude_from_sim no)
+		(at 134.6161 98.806 0)
+		(effects
+			(font
+				(size 1.27 1.27)
+			)
+			(justify left bottom)
+		)
+	)
+	(text "0x02 hw_version"
+		(exclude_from_sim no)
+		(at 134.874 101.346 0)
+		(effects
+			(font
+				(size 1.27 1.27)
+			)
+			(justify left bottom)
+		)
+	)
 	(text "JLC alternatives\n\n| jlc | USD/Stock | Package | Comments |\n| - | - | - | - |\n| C2831468  | 0.37/1k  | SMD2520-4P | 1nd |\n| C2901596  | 0.37/1k  | SMD2520-4P | 2nd |\n| C437139   | 0.29/188 | SMD2520-4P | 2nd |\n| C387449   | 0.49/3k  | SMD2520-4P | 2nd |\n| C409301   | 0.55/2k  | SMD2520-4P | 2nd |"
 		(exclude_from_sim no)
@@
 	)
 	(junction
-		(at 132.08 101.6)
-		(diameter 0)
-		(color 0 0 0 0)
-	)
-	(junction
-		(at 129.54 93.98)
-		(diameter 0)
-		(color 0 0 0 0)
-	)
-	(junction
 		(at 102.87 30.48)
 		(diameter 1.016)
@@
 	(wire
 		(pts
-			(xy 134.62 101.6) (xy 132.08 101.6)
-		)
-		(stroke
-			(width 0)
-			(type default)
-		)
-	)
-	(wire
-		(pts
 			(xy 44.45 48.26) (xy 53.34 48.26)
 		)
@@
 	(wire
 		(pts
-			(xy 134.62 96.52) (xy 129.54 96.52)
-		)
-		(stroke
-			(width 0)
-			(type default)
-		)
-	)
-	(wire
-		(pts
 			(xy 88.9 124.46) (xy 88.9 121.92)
 		)
@@
 	(wire
 		(pts
-			(xy 134.62 93.98) (xy 129.54 93.98)
-		)
-		(stroke
-			(width 0)
-			(type default)
-		)
-	)
-	(wire
-		(pts
 			(xy 49.53 104.14) (xy 49.53 115.57)
 		)
@@
 	(wire
 		(pts
-			(xy 134.62 99.06) (xy 129.54 99.06)
-		)
-		(stroke
-			(width 0)
-			(type default)
-		)
-	)
-	(wire
-		(pts
 			(xy 129.54 96.52) (xy 129.54 99.06)
 		)
@@
 	(wire
 		(pts
-			(xy 129.54 104.14) (xy 134.62 104.14)
-		)
-		(stroke
-			(width 0)
-			(type default)
-		)
-	)
-	(wire
-		(pts
 			(xy 162.56 33.02) (xy 162.56 31.75)
 		)
@@
 		)
 	)
-	(label "HW_VERSION_1"
-		(at 134.62 101.6 0)
-		(effects
-			(font
-				(size 1.27 1.27)
-				(italic yes)
-			)
-			(justify left bottom)
-		)
-	)
 	(label "QSPI_SD2"
 		(at 135.89 76.2 180)
@@
 		)
 	)
-	(label "HW_VERSION_2"
-		(at 134.62 99.06 0)
-		(effects
-			(font
-				(size 1.27 1.27)
-				(italic yes)
-			)
-			(justify left bottom)
-		)
-	)
 	(label "QSPI_SCLK"
 		(at 247.65 97.79 180)
@@
 		)
 	)
-	(label "HW_VERSION_3"
-		(at 134.62 96.52 0)
-		(effects
-			(font
-				(size 1.27 1.27)
-				(italic yes)
-			)
-			(justify left bottom)
-		)
-	)
 	(label "+1V1"
 		(at 182.88 27.94 0)
@@
 		)
 	)
-	(label "HW_VERSION_0"
-		(at 134.62 104.14 0)
-		(effects
-			(font
-				(size 1.27 1.27)
-				(italic yes)
-			)
-			(justify left bottom)
-		)
-	)
 	(label "QSPI_SS"
 		(at 247.65 95.25 180)
@@
 		)
 	)
-	(label "HW_VERSION_4"
-		(at 134.62 93.98 0)
-		(effects
-			(font
-				(size 1.27 1.27)
-				(italic yes)
-			)
-			(justify left bottom)
-		)
-	)
 	(label "LED_ACTIVE"
 		(at 184.15 135.89 0)
@@
 			)
 		)
-		(property "Value" "27R"
+		(property "Value" "33R"
 			(at 128.27 89.0016 90)
 			(effects
@@
 			)
 		)
-		(property "Value" "27R"
+		(property "Value" "33R"
 			(at 128.27 86.4616 90)
 			(effects
