File: kicad/octohub4_v0.1/pcb_octoprobe.kicad_pcb (KiCad board)
At the start: 2 copper layers, 100 x 165 mm, 955 parts, among them J1302 Conn_02x20, J1303 Conn_02x20, J1501 Conn_02x20, J1502 Conn_01x12, J201 Conn_02x05, J202 Conn_01x5, J301 USB_C_Receptacle_USB2.0, J501 Conn_02x20, U1001 GAQY221S, U1101 GAQY221S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

Commit message: KiCad cleanup
Parts:
- removed BP201, BP202: octoprobe_prototype_board, 00_project_library:octoprobe_breakout_PB
- removed C1501, C1502, C1505, C1506, C1507, C1508, C1509, C1510, C1511, C1512, C203, C204, C207, C208, C209, C210, C211, C212, C213, C214: 100n, Capacitor_SMD:C_0402_1005Metric
- removed C1503, C1504, C205, C206, C217: 1u, Capacitor_SMD:C_0402_1005Metric
- removed C201, C202, C215: 10u, Capacitor_SMD:C_0603_1608Metric
- removed C216: 1000u, Capacitor_THT:CP_Radial_D8.0mm_P2.50mm
- removed D103, D104: green, LED_SMD:LED_0805_2012Metric
- removed D1501, D202: B5819W SL, Diode_SMD:D_SOD-123
- removed D1502, D1503: white, 00_project_library:LED_0603_1608Metric
- removed H1308: octoprobe_MountingHole, MountingHole:MountingHole_3.2mm_M3_DIN965_Pad
- removed J1501: Conn_02x20, 00_project_library:PinSocket_2x12_P2.54mm_Vertical_squarepad
- removed J1502: Conn_01x12, 00_project_library:PinSocket_1x12_P2.54mm_Vertical_squarepad
- removed R103, R104: 4K7, Resistor_SMD:R_0805_2012Metric
- removed R1501, R1502, R202, R203: 33R, Resistor_SMD:R_0402_1005Metric
- removed R1503, R205: 0R, Resistor_SMD:R_0805_2012Metric
- removed R1504, R207, R210, R213: 10K, Resistor_SMD:R_0402_1005Metric
- removed R1505: 100K, Resistor_SMD:R_0402_1005Metric
- removed R1506, R1507: 2k2, Resistor_SMD:R_0402_1005Metric
- removed R1508: 10k, Resistor_SMD:R_0402_1005Metric
- removed R201, R204: 1K, Resistor_SMD:R_0805_2012Metric
- removed R208: 2K7, Resistor_SMD:R_0603_1608Metric
- removed R209: 3K6, Resistor_SMD:R_0603_1608Metric
- removed R211: 100k, Resistor_SMD:R_0402_1005Metric
- removed R212: 33K, Resistor_SMD:R_0402_1005Metric
- removed U1501, U201: RP2040, 00_project_library:RP2040-QFN-56
- removed U1502, U203: W25Q32JVS, 00_project_library:SOIC-8_5.23x5.23mm_P1.27mm
- removed U1503, U1504: TXB0108PW, Package_SO:TSSOP-20_4.4x6.5mm_P0.65mm
- removed U202: AMS1117-3.3, 00_project_library:SOT-223-3_TabPin2
- removed U204, U205, U207: TPS2595xx, Package_SON:WSON-8-1EP_2x2mm_P0.5mm_EP0.9x1.6mm
- removed X201: Oscillator-12MHz, Crystal:Crystal_SMD_2520-4Pin_2.5x2.0mm
Routing:
- net (no net): track 0.00 -> 2219.6 mm, vias 2 -> 55
- net /RP2 CPU/LED_ACTIVE: track 253.2 -> 0.00 mm
- net Net-(D103-A): track 251.0 -> 0.00 mm
- net /RP2 CPU/LED_ERR: track 218.6 -> 0.00 mm
- net RP2_PROBE_RUN: track 66.7 -> 0.00 mm, vias 2 -> 0
- net /RP2 CPU/12MHz: track 58.7 -> 0.00 mm, vias 5 -> 0
- net /RP2 PROBE/GPIO3: track 48.0 -> 0.00 mm, vias 2 -> 0
- net /RP2 PROBE/GPIO2: track 47.7 -> 0.00 mm, vias 3 -> 0
- net /RP2 PROBE/GPIO4: track 44.7 -> 0.00 mm, vias 3 -> 0
- net RP2_PROBE_BOOT: track 43.4 -> 0.00 mm, vias 2 -> 0
- net /RP2 PROBE/GPIO28: track 43.1 -> 0.00 mm
- net /RP2 PROBE/GPIO5: track 42.1 -> 0.00 mm, vias 2 -> 0
- net /RP2 PROBE/VDUT: track 40.8 -> 0.00 mm
- net /RP2 PROBE/GPIO26: track 40.3 -> 0.00 mm
- net /RP2 PROBE/GPIO10: track 39.1 -> 0.00 mm, vias 3 -> 0
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