File: kicad/octohub4_v0.1/pcb_octoprobe.kicad_sch (KiCad schematic)
At the start: 10 parts, among them J202 Conn_01x5

Commit message: KiCad cleanup
Other:
- removed sheet Prototype Area
- removed sheet RP2 CPU
- removed sheet RP2 PROBE
- removed sheet Regulator 3V3
- removed sheet Relay Breakout
- title: Octoprobe tentacle -> Octohub4
