File: kicad/octohub4_v0.1/pcb_octoprobe_cpu.kicad_sch (KiCad schematic)
At the start: 27 parts, among them J201 Conn_02x05, U201 RP2040, U203 W25Q32JVS, X201 Oscillator-12MHz

Commit message: KiCad cleanup
Other:
- title: Octoprobe tentacle -> Octohub4
Changed lines of the file:
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@@
 	(paper "A4")
 	(title_block
-		(title "Octoprobe tentacle")
-		(date "2025-11-24")
-		(rev "0.6")
+		(title "Octohub4")
+		(date "2026-01-11")
+		(rev "0.1")
 		(company "Hans Märki, Märki Informatik")
 		(comment 1 "The MIT License (MIT)")
