File: kicad/octohub4_v0.1/pcb_octoprobe_usbhubchip.kicad_sch (KiCad schematic)
At the start: 34 parts, among them J301 USB_C_Receptacle_USB2.0, U302 USB2514B_Bi, Y301 24MHz

Commit message: KiCad cleanup
Other:
- title: Octoprobe tentacle -> Octohub4
Changed lines of the file:
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@@
 	(paper "A4")
 	(title_block
-		(title "Octoprobe tentacle")
-		(date "2025-11-24")
-		(rev "0.6")
+		(title "Octohub4")
+		(date "2026-01-11")
+		(rev "0.1")
 		(company "Hans Märki, Märki Informatik")
 		(comment 1 "The MIT License (MIT)")
