File: kicad/octohub4_v0.1/pcb_octohub4.kicad_pcb (KiCad board)
At the start: 2 copper layers, 100 x 165 mm, 882 parts, among them J1302 Conn_02x20, J1303 Conn_02x20, J201 Conn_02x05, J202 Conn_01x5, J301 USB_C_Receptacle_USB2.0, J501 Conn_02x20, U1001 GAQY221S, U1101 GAQY221S, U1201 GAQY221S, U302 USB2514B_Bi, U601 GAQY221S, U701 GAQY221S, U801 GAQY221S, U901 GAQY221S, Y301 24MHz

Commit message: Collecting components
Parts:
- removed ? (x772): prototype_NC, 00_project_library:octoprobe_breakout_PB_NC
- removed ? (x20): prototype_GND, 00_project_library:octoprobe_breakout_PB
- removed D1001, D1101, D1201, D601, D701, D801, D901: white, 00_project_library:LED_0603_1608Metric
- removed D201: blue, LED_SMD:LED_0805_2012Metric
- removed D203: red, 00_project_library:LED_0603_1608Metric
- removed H1305, H1306, H1307: octoprobe_MountingHole, MountingHole:MountingHole_3.2mm_M3_DIN965_Pad
- removed J1302, J1303: Conn_02x20, 00_project_library:PinSocket_2x20_P2.54mm_Vertical-stackable_squarepad
- removed J501: Conn_02x20, 00_project_library:PinSocket_2x14_P2.54mm_Vertical_squarepad
- removed R1001, R1101, R1201, R601, R701, R801, R901: 2k2, Resistor_SMD:R_0805_2012Metric
- removed R1002, R1102, R1202, R602, R702, R802, R902: 390, Resistor_SMD:R_0805_2012Metric
- removed U1001, U1101, U1201, U601, U701, U801, U901: GAQY221S, 00_project_library:SOP-4_4.4x4.3mm_P2.54mm
- removed UR1001: 5, 00_project_library:octoprobe_relay
- removed UR1101: 6, 00_project_library:octoprobe_relay
- removed UR1201: 7, 00_project_library:octoprobe_relay
- removed UR601: 1, 00_project_library:octoprobe_relay
- removed UR701: 2, 00_project_library:octoprobe_relay
- removed UR801: 3, 00_project_library:octoprobe_relay
- removed UR901: 4, 00_project_library:octoprobe_relay
- added H201: MountingHole_Pad, 00_project_library:octohub4_mounting_hole, F.Cu at (64.8, 23.3)
- added H202: MountingHole_Pad, 00_project_library:octohub4_mounting_hole, F.Cu at (152.8, 23.3)
- added H203: MountingHole_Pad, 00_project_library:octohub4_mounting_hole, F.Cu at (64.8, 91.3)
- added H204: MountingHole_Pad, 00_project_library:octohub4_mounting_hole, F.Cu at (152.8, 91.3)
- added J101: USB-231-ARY, 00_project_library:USB231ARY, F.Cu at (83.0, 30.1)
- added J102: USB-231-ARY, 00_project_library:USB231ARY, F.Cu at (102.3, 30.1)
- added J103: USB-231-ARY, 00_project_library:USB231ARY, F.Cu at (121.6, 30.1)
- added J104: USB-231-ARY, 00_project_library:USB231ARY, F.Cu at (140.8, 30.1)
- added J203: Barrel_Jack_Switch, 00_project_library:BarrelJack_D5.5mm, F.Cu at (69.2, 80.2)
- added U201: RPW0010A-MFG, 00_project_library:TPS259474LRPWR, F.Cu at (83.6, 82.1)
- J201: value Conn_02x05 -> Screw_Terminal_01x02; footprint 00_project_library:PinSocket_2x05_P2.54mm_Vertical_squarepad -> 00_project_library:KF235-2P
- moved BP203 197.5 mm to (-44.2, 45.4)
- moved C303 189.2 mm to (-67.6, 82.6)
- moved C305 189.2 mm to (-65.3, 77.7)
- moved C308 189.2 mm to (-72.3, 82.1)
- moved NT102 189.2 mm to (-46.8, 99.8)
- moved NT301 189.2 mm to (-94.2, 74.8)
- moved R302 189.2 mm to (-98.7, 83.5)
- moved R305 189.2 mm to (-67.7, 77.6)
- moved R306 189.2 mm to (-65.5, 80.3)
- moved Y301 189.2 mm to (-72.3, 85.2)
- moved C301 189.2 mm to (-68.1, 88.2)
- moved C302 189.2 mm to (-57.7, 87.1)
- moved C304 189.2 mm to (-62.0, 79.8)
- moved C306 189.2 mm to (-66.7, 77.6)
- moved C307 189.2 mm to (-72.3, 88.4)
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Connections:
- J201 pad 1: Net-(J201-Pin_1) -> unconnected-(J201-Pin_1-Pad1)
- J201 pad 2: Net-(J201-Pin_2) -> unconnected-(J201-Pin_2-Pad2)
Routing:
- net (no net): track 2219.6 -> 231.5 mm, vias 55 -> 10
- net +3V3infra: track 429.1 -> 0.00 mm, vias 6 -> 0
- net GND: track 160.6 -> 16.7 mm, vias 467 -> 135
- net +5Vbuf: track 95.6 -> 0.00 mm, vias 4 -> 0
- net Net-(J201-Pin_8): track 60.3 -> 0.00 mm
- net Net-(J201-Pin_6): track 49.2 -> 0.00 mm
- net Net-(J201-Pin_7): track 46.4 -> 0.00 mm, vias 2 -> 0
- net Net-(J201-Pin_5): track 43.8 -> 0.00 mm, vias 2 -> 0
- net Net-(J201-Pin_4): track 43.7 -> 0.00 mm
- net Net-(J201-Pin_2): track 42.1 -> 0.00 mm
- net Net-(J201-Pin_3): track 40.8 -> 0.00 mm, vias 2 -> 0
- net RP2_INFRA_BOOT: track 75.9 -> 36.9 mm, vias 2 -> 1
- net Net-(J201-Pin_1): track 38.6 -> 0.00 mm, vias 2 -> 0
- net RELAIS_1: track 31.9 -> 0.00 mm
- net RELAIS_2: track 27.3 -> 0.00 mm
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- removed copper zone on B.Cu, net GND
Other:
- board size 100 x 165 mm -> 100 x 80 mm
- board text added: "Octoprobe octohub4"
- board text removed: "(blue)"
- board text removed: "(red)"
- board text removed: "1"
- board text removed: "10"
- board text removed: "11"
- board text removed: "12"
- board text removed: "13"
- board text removed: "14"
- board text removed: "15"
- board text removed: "16"
- board text removed: "17"
- board text removed: "18"
- board text removed: "19"
- board text removed: "2"
- board text removed: "20"
- board text removed: "21"
- board text removed: "22"
- board text removed: "23"
- board text removed: "24"
- board text removed: "25"
- board text removed: "26"
- board text removed: "27"
- board text removed: "28"
- board text removed: "29"
- board text removed: "3"
- board text removed: "30"
- board text removed: "31"
- board text removed: "32"
- board text removed: "33"
- board text removed: "34"
- board text removed: "35"
- board text removed: "36"
- board text removed: "37"
- board text removed: "38"
- board text removed: "39"
- board text removed: "4"
- board text removed: "40"
- board text removed: "5"
- board text removed: "6"
- board text removed: "7"
- board text removed: "8"
- board text removed: "9"
- board text removed: "Active"
- board text removed: "DUT"
- board text removed: "DUT USB"
- board text removed: "DUT<3V3"
- board text removed: "DUT>3V3"
- board text removed: "Device Under Test Power (green)"
- board text removed: "Error"
- board text removed: "GND"
- board text removed: "Infra"
- board text removed: "Infrastructure (green) Power"
- board text removed: "OCTOBUS_"
- board text removed: "Octoprobe tentacle"
- board text removed: "PICO_INFRA"
- board text removed: "PICO_PROBE"
- board text removed: "Run"
- board text removed: "level shifter"
- board text removed: "serial"
- board text removed: "www.github.com/octoprobe/tentacle"

Commit message: Collecting components 2
Parts:
- NT101, NT102, NT103, NT104, NT105, NT106, NT301, NT302: value octoprobe_NetTie_USB_Differential -> NetTie-4_USB_Differential

Commit message: Collecting components 3
Parts:
- J101, J102, J103, J104: value USB-231-ARY -> USB231ARY
- NT101, NT102, NT103, NT104, NT105, NT106, NT301, NT302: value NetTie-4_USB_Differential -> octoprobe_NetTie_USB_Differential
- U201: value RPW0010A-MFG -> TPS259474LRPWR
- moved J201 5.82 mm to (63.8, 62.3), turned to 90 degrees
Connections:
- J201 pad 1: unconnected-(J201-Pin_1-Pad1) -> +5V
- J201 pad 2: unconnected-(J201-Pin_2-Pad2) -> GND
- J203 pad 1: unconnected-(J203-Pad1) -> +5V
- J203 pad 2: unconnected-(J203-Pad2) -> GND
- J203 pad 3: unconnected-(J203-Pad3) -> GND

Commit message: tmp
Parts:
- removed D101: white, 00_project_library:LED_0603_1608Metric
- removed J202: Conn_01x5, 00_project_library:PinSocket_1x5_P2.54mm_Vertical_squarepad_USB
- removed R101: 2k2, Resistor_SMD:R_0805_2012Metric
- added BP201: Solder 5V, Connector_Wire:SolderWirePad_1x01_SMD_2x4mm, F.Cu at (27.1, -3.96)
- added BP202: Solder GND, Connector_Wire:SolderWirePad_1x01_SMD_2x4mm, F.Cu at (27.1, 0.38)
- added BP204: Scope 5V OUT, 00_project_library:octoprobe_breakout_PB, F.Cu at (-108.1, 109.3)
- added BP205: Scope 5V IN, 00_project_library:octoprobe_breakout_PB, F.Cu at (-104.0, 109.3)
- added C201: 100n, Capacitor_SMD:C_0402_1005Metric, F.Cu at (113.8, -17.8)
- added C202: 100n, Capacitor_SMD:C_0402_1005Metric, F.Cu at (113.8, -15.8)
- added C203: 100n, Capacitor_SMD:C_0402_1005Metric, F.Cu at (113.8, -13.8)
- added C216: 1000u, Capacitor_THT:CP_Radial_D8.0mm_P2.50mm, F.Cu at (105.3, -3.24)
- added C311: 10u, Capacitor_SMD:C_0603_1608Metric, F.Cu at (-115.9, 105.3)
- added C312: 10u, Capacitor_SMD:C_0603_1608Metric, F.Cu at (70.8, 63.6)
- added H1301: octoprobe_CableTieHole, 00_project_library:octoprobe_CableTieHole, F.Cu at (14.3, -4.29)
- added H1302: octoprobe_CableTieHole, 00_project_library:octoprobe_CableTieHole, F.Cu at (14.3, 0.76)
- added H201: MountingHole_Pad, 00_project_library:octohub4_mounting_hole, F.Cu at (64.8, 23.3)
- added H202: MountingHole_Pad, 00_project_library:octohub4_mounting_hole, F.Cu at (152.8, 23.3)
- added H203: MountingHole_Pad, 00_project_library:octohub4_mounting_hole, F.Cu at (64.8, 91.3)
- added H204: MountingHole_Pad, 00_project_library:octohub4_mounting_hole, F.Cu at (152.8, 91.3)
- added NT107: octoprobe_NetTie_USB_Differential, 00_project_library:octoprobe_NetTie_USB_Differential, F.Cu at (170.3, 70.2)
- added NT108: octoprobe_NetTie_USB_Differential, 00_project_library:octoprobe_NetTie_USB_Differential, F.Cu at (170.3, 72.8)
- added R201: 137, Resistor_SMD:R_0805_2012Metric, F.Cu at (117.4, -17.3)
- added U301: AMS1117-3.3, 00_project_library:SOT-223-3_TabPin2, F.Cu at (71.0, 57.1)
- moved NT106 241.8 mm to (170.3, 67.7), turned to 0 degrees
- moved NT103 238.0 mm to (170.3, 62.5), turned to 0 degrees
- moved NT105 234.4 mm to (170.3, 65.1), turned to 0 degrees
- moved NT101 233.0 mm to (170.3, 57.4), turned to 0 degrees
- moved NT102 220.8 mm to (170.3, 60.0), turned to 0 degrees
- moved C401 174.6 mm to (68.9, 73.4), turned to 180 degrees
- moved R304 174.5 mm to (110.3, 59.3)
- moved R305 174.5 mm to (105.8, 59.3)
- moved R308 174.5 mm to (112.5, 61.4)
- moved R312 174.5 mm to (115.8, 67.8)
- moved C301 174.5 mm to (105.5, 69.9)
- moved C302 174.5 mm to (115.8, 68.8)
- moved C303 174.5 mm to (105.9, 64.2)
- moved C304 174.5 mm to (111.5, 61.4)
- moved C305 174.5 mm to (108.2, 59.3)
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Connections:
- net RP2_INFRA_PWR_EN renamed /USB Hub Chip/PRT_PWR1
- C401 pad 2: HUB+5V -> +5VIN
- D302 pad 5: HUB+5V -> +5VIN
- J101 pad 1: unconnected-(J101-VBUS-Pad1) -> +5VOUT
- J101 pad 2: unconnected-(J101-D--Pad2) -> Net-(J101-D-)
- J101 pad 3: unconnected-(J101-D+-Pad3) -> Net-(J101-D+)
- J101 pad 4: unconnected-(J101-GND-Pad4) -> GND
- J101 pad MH: unconnected-(J101-PadMH) -> GND
- J102 pad 1: unconnected-(J102-VBUS-Pad1) -> +5VOUT
- J102 pad 2: unconnected-(J102-D--Pad2) -> Net-(J102-D-)
- J102 pad 3: unconnected-(J102-D+-Pad3) -> Net-(J102-D+)
- J102 pad 4: unconnected-(J102-GND-Pad4) -> GND
- J102 pad MH: unconnected-(J102-PadMH) -> GND
- J103 pad 1: unconnected-(J103-VBUS-Pad1) -> +5VOUT
- J103 pad 2: unconnected-(J103-D--Pad2) -> Net-(J103-D-)
- J103 pad 3: unconnected-(J103-D+-Pad3) -> Net-(J103-D+)
- J103 pad 4: unconnected-(J103-GND-Pad4) -> GND
- J103 pad MH: unconnected-(J103-PadMH) -> GND
- J104 pad 1: unconnected-(J104-VBUS-Pad1) -> +5VOUT
- J104 pad 2: unconnected-(J104-D--Pad2) -> Net-(J104-D-)
- J104 pad 3: unconnected-(J104-D+-Pad3) -> Net-(J104-D+)
- J104 pad 4: unconnected-(J104-GND-Pad4) -> GND
- J104 pad MH: unconnected-(J104-PadMH) -> GND
- J201 pad 1: +5V -> +5VIN
- J203 pad 1: +5V -> +5VIN
- J301 pad A4: HUB+5V -> +5VIN
- J301 pad A9: HUB+5V -> +5VIN
- J301 pad B4: HUB+5V -> +5VIN
- J301 pad B9: HUB+5V -> +5VIN
- NT101 pad 1: /USB Hub Chip/USB_DP4 -> /USB Hub Chip/USB_DP1
- NT101 pad 3: /USB Hub Chip/USB_DM4 -> /USB Hub Chip/USB_DM1
- NT102 pad 1: _USB_PROBE_D- -> Net-(J101-D-)
- NT102 pad 3: _USB_PROBE_D+ -> Net-(J101-D+)
- NT103 pad 1: /USB Hub Chip/USB_DP1 -> /USB Hub Chip/USB_DP2
- NT103 pad 3: /USB Hub Chip/USB_DM1 -> /USB Hub Chip/USB_DM2
- NT104 pad 1: _USB_INFRA_D- -> Net-(J102-D-)
- NT104 pad 3: _USB_INFRA_D+ -> Net-(J102-D+)
- NT106 pad 1: Net-(J202-Pin_2) -> Net-(J103-D-)
- NT106 pad 3: Net-(J202-Pin_3) -> Net-(J103-D+)
- R301 pad 2: HUB+5V -> +5VOUT
- R305 pad 2: HUB+5V -> +5VOUT
- U201 pad 1: unconnected-(U201-EN_UVLO-Pad1) -> +5VIN
- U201 pad 10: unconnected-(U201-ITIMER-Pad10) -> Net-(U201-ITIMER)
- U201 pad 2: unconnected-(U201-OVCSEL-Pad2) -> GND
- U201 pad 5: unconnected-(U201-IN-Pad5) -> +5VIN
- U201 pad 6: unconnected-(U201-OUT-Pad6) -> +5VOUT
- U201 pad 7: unconnected-(U201-dVdt-Pad7) -> Net-(U201-dVdt)
- U201 pad 8: unconnected-(U201-GND-Pad8) -> GND
- U201 pad 9: unconnected-(U201-ILM-Pad9) -> Net-(U201-ILM)
- U302 pad 16: RP2_INFRA_BOOT -> /USB Hub Chip/PRT_PWR2
Routing:
- net (no net): track 231.5 -> 77.5 mm, vias 10 -> 1
- net HUB+5V: track 68.0 -> 0.00 mm, vias 2 -> 0
- net /USB Hub Chip/PRT_PWR2: track 0.00 -> 36.9 mm, vias 0 -> 1
- net RP2_INFRA_BOOT: track 36.9 -> 0.00 mm, vias 1 -> 0
- net +5VOUT: track 0.00 -> 33.3 mm, vias 0 -> 2
- net /USB_INFRA_D+: track 29.2 -> 0.00 mm
- net /USB_INFRA_D-: track 28.9 -> 0.00 mm
- net /USB Hub Chip/USB_UP_D-: track 25.0 -> 6.20 mm
- net /USB Hub Chip/USB_UP_D+: track 24.2 -> 5.84 mm
- net +3V3: track 89.6 -> 72.0 mm, vias 6 -> 5
- net /USB_PROBE_D-: track 14.7 -> 0.00 mm
- net /USB_PROBE_D+: track 14.7 -> 0.00 mm
- net /USB_DUT_D+: track 12.7 -> 0.00 mm
- net /USB_DUT_D-: track 12.4 -> 0.00 mm
- net +5Vdut: track 11.6 -> 0.00 mm, vias 2 -> 0
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Other:
- board text removed: "5V"
- board text removed: "Boot"
- board text removed: "DUT_PWR_EN"

Commit message: Add run_kicad_purge 2
Parts:
- removed the H201 at (64.8, 23.3) (x2)
- removed the H202 at (152.8, 23.3) (x2)
- removed the H203 at (64.8, 91.3)
- removed the H204 at (152.8, 91.3) (x2)
- added D201: SS34, Diode_SMD:D_SMA, F.Cu at (76.7, 74.0)
- added D202: SS34, Diode_SMD:D_SMA, F.Cu at (76.7, 70.5)
- added D203: PRTR5V0U2X, Package_SON:Texas_USON-6_1x1.45mm_P0.5mm_SMD, F.Cu at (78.2, 80.5)
- added D204: PRTR5V0U2X, Package_SON:Texas_USON-6_1x1.45mm_P0.5mm_SMD, F.Cu at (98.1, 80.5)
- added D205: PRTR5V0U2X, Package_SON:Texas_USON-6_1x1.45mm_P0.5mm_SMD, F.Cu at (120.7, 80.5)
- added D206: PRTR5V0U2X, Package_SON:Texas_USON-6_1x1.45mm_P0.5mm_SMD, F.Cu at (140.2, 80.5)
- added H201: MountingHole_Pad, 00_project_library:octohub4_mounting_hole, F.Cu at (64.8, 23.3)
- added H202: MountingHole_Pad, 00_project_library:octohub4_mounting_hole, F.Cu at (152.8, 23.3)
- added H204: MountingHole_Pad, 00_project_library:octohub4_mounting_hole, F.Cu at (152.8, 91.3)
- added JP201: SolderJumper_2_Bridged, Jumper:SolderJumper-2_P1.3mm_Bridged_RoundedPad1.0x1.5mm, F.Cu at (71.8, 23.3)
- added JP202: SolderJumper_2_Bridged, Jumper:SolderJumper-2_P1.3mm_Bridged_RoundedPad1.0x1.5mm, F.Cu at (146.1, 23.3)
- added JP203: SolderJumper_2_Open, Jumper:SolderJumper-2_P1.3mm_Open_RoundedPad1.0x1.5mm, F.Cu at (83.5, 74.0)
- added JP204: SolderJumper_2_Bridged, Jumper:SolderJumper-2_P1.3mm_Bridged_RoundedPad1.0x1.5mm, F.Cu at (83.4, 70.5)
- added JP205: SolderJumper_2_Open, Jumper:SolderJumper-2_P1.3mm_Open_RoundedPad1.0x1.5mm, F.Cu at (124.1, 62.9)
- moved BP203 245.7 mm to (129.8, 50.7)
- moved BP204 243.8 mm to (129.8, 55.8)
- moved BP205 240.4 mm to (129.8, 53.2)
- moved C311 189.9 mm to (71.2, 73.1), turned to -90 degrees
- moved NT104 125.0 mm to (100.8, 81.6), turned to 45 degrees
- moved NT102 91.8 mm to (81.1, 81.6), turned to 45 degrees
- moved C202 85.3 mm to (132.0, 67.5)
- moved R201 84.4 mm to (131.2, 66.0), turned to 180 degrees
- moved C201 82.2 mm to (120.9, 64.1), turned to -90 degrees
- moved C203 80.5 mm to (132.0, 64.5)
- moved U201 79.7 mm to (124.5, 66.8)
- moved BP201 79.6 mm to (92.5, 41.4)
- moved BP202 79.6 mm to (92.5, 45.7)
- moved H1301 79.6 mm to (79.8, 41.0)
- moved H1302 79.6 mm to (79.8, 46.1)
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Connections:
- net /USB_INFRA_D+ renamed /USB_2_D+
- net /USB_INFRA_D- renamed /USB_2_D-
- net /USB_PROBE_D+ renamed /USB_1_D+
- net /USB_PROBE_D- renamed /USB_1_D-
- BP204 pad 1: +5VOUT -> +5VPROTECTED
- C216 pad 1: +5VOUT -> +5VPROTECTED
- C311 pad 1: +5VOUT -> Net-(D201-K)
- C401 pad 2: +5VIN -> +5VUPSTREAM
- D302 pad 5: +5VIN -> +5VUPSTREAM
- J101 pad 1: +5VOUT -> +5VPROTECTED
- J102 pad 1: +5VOUT -> +5VPROTECTED
- J103 pad 1: +5VOUT -> +5VPROTECTED
- J104 pad 1: +5VOUT -> +5VPROTECTED
- J301 pad A4: +5VIN -> +5VUPSTREAM
- J301 pad A9: +5VIN -> +5VUPSTREAM
- J301 pad B4: +5VIN -> +5VUPSTREAM
- J301 pad B9: +5VIN -> +5VUPSTREAM
- NT105 pad 2: /USB_DUT_D+ -> /USB_3_D+
- NT105 pad 4: /USB_DUT_D- -> /USB_3_D-
- NT106 pad 2: /USB_DUT_D- -> /USB_3_D-
- NT106 pad 4: /USB_DUT_D+ -> /USB_3_D+
- NT107 pad 2: /USB_DUT_D+ -> /USB_4_D+
- NT107 pad 4: /USB_DUT_D- -> /USB_4_D-
- NT108 pad 2: /USB_DUT_D- -> /USB_4_D-
- NT108 pad 4: /USB_DUT_D+ -> /USB_4_D+
- R301 pad 2: +5VOUT -> +5VUPSTREAM
- R305 pad 2: +5VOUT -> +5VUPSTREAM
- U201 pad 6: +5VOUT -> +5VPROTECTED
- U301 pad 3: +5VOUT -> Net-(D201-K)
Routing:
- net +5VIN: track 0.00 -> 280.8 mm
- net +5VPROTECTED: track 0.00 -> 209.1 mm, vias 0 -> 7
- net +5VUPSTREAM: track 0.00 -> 84.4 mm, vias 0 -> 4
- net (no net): track 77.5 -> 0.00 mm, vias 1 -> 0
- net /USB Hub Chip/PRT_PWR2: track 36.9 -> 2.57 mm
- net +5VOUT: track 33.3 -> 0.00 mm, vias 2 -> 0
- net +3V3: track 72.0 -> 99.4 mm
- net /USB_4_D-: track 0.00 -> 25.1 mm
- net /USB_4_D+: track 0.00 -> 25.1 mm
- net /USB_1_D-: track 0.00 -> 25.0 mm
- net /USB_1_D+: track 0.00 -> 24.9 mm
- net /USB Hub Chip/USB_UP_D+: track 5.84 -> 25.5 mm
- net /USB Hub Chip/USB_UP_D-: track 6.20 -> 25.7 mm
- net Net-(D201-K): track 0.00 -> 11.6 mm
- net /USB_2_D+: track 0.00 -> 7.93 mm
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- added copper zone on B.Cu, net GND
Other:
- board text added: "5V in"
- board text added: "5V protected"
- board text added: "GND"
- board text removed: "Scope GND"

Commit message: Add run_kicad_purge 3
Parts:
- added D207: green, LED_SMD:LED_0805_2012Metric, F.Cu at (131.1, 73.3)
- added R202: 4K7, Resistor_SMD:R_0805_2012Metric, F.Cu at (127.0, 73.3)
- moved D301 21.6 mm to (75.7, 61.8)
- moved R301 21.6 mm to (72.0, 61.8)
- moved BP202 17.5 mm to (89.8, 28.5)
- moved H1301 14.8 mm to (73.3, 27.8)
- moved H1302 14.8 mm to (73.3, 32.8)
- moved C216 11.8 mm to (150.4, 75.6), turned to 0 degrees
- moved BP201 9.79 mm to (89.8, 32.0)
- moved J203 5.60 mm to (69.3, 44.7)
- moved Logo_open_hardware101 4.89 mm to (149.7, 41.2)
- moved BP204 2.58 mm to (129.8, 58.3)
- moved BP203 2.58 mm to (129.8, 53.3)
- moved BP205 2.58 mm to (129.8, 55.8)
- moved D201 1.20 mm to (75.5, 74.0)
- moved D202 1.20 mm to (75.5, 70.5)
- moved JP203 1.20 mm to (82.3, 74.0)
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Connections:
- J201 pad 1: +5VIN -> GND
- J201 pad 2: GND -> +5VIN
Routing:
- net +5VIN: track 280.8 -> 255.8 mm
- net +5VUPSTREAM: track 84.4 -> 61.7 mm
- net +5VPROTECTED: track 209.1 -> 205.7 mm, vias 7 -> 6
- net Net-(D201-K): track 11.6 -> 8.69 mm
- net /USB Hub Chip/PRT_PWR2: track 2.57 -> 0.00 mm, vias 1 -> 0
- net Net-(D207-A): track 0.00 -> 2.21 mm
- net GND: track 13.1 -> 15.0 mm, vias 36 -> 55
- net Net-(D301-A): track 0.00 -> 1.83 mm
- net /USB Hub Chip/PRT_PWR1: track 1.31 -> 0.00 mm, vias 1 -> 0
- net Net-(D302-I/O2-Pad3): track 8.14 -> 9.19 mm
- net Net-(D302-I/O1-Pad1): track 7.99 -> 8.93 mm
- net Net-(J102-D+): track 4.40 -> 5.26 mm
- net Net-(U201-ILM): track 5.98 -> 5.14 mm
- net Net-(J103-D-): track 6.32 -> 6.92 mm
- net Net-(J104-D+): track 6.93 -> 7.50 mm
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Other:
- board text added: "+5V IN"
- board text added: "+5V PROTECTED"
- board text added: "+5V UPSTREAM"
- board text added: "1"
- board text added: "2"
- board text added: "3"
- board text added: "4"
- board text added: "5V IN"
- board text added: "5V IN Barrel Jack"
- board text added: "5V PROTECTED"
- board text added: "5V PROTECTED USB-A 1,2,3,4"
- board text added: "5V UPSTREAM USB-C"
- board text added: "5V power distribution"
- board text added: "Barrel Jack"
- board text added: "Clamp Terminal"
- board text added: "POWER +5V PROTECTED"
- board text added: "POWER +5V UPSTREAM"
- board text added: "Solder Pads"
- board text added: "USB HUB"
- board text added: "center: +5V IN"
- board text removed: "5V in"
- board text removed: "5V protected"
- board text removed: "Infrastructure"
- board text removed: "Octoprobe octohub4"
- board text removed: "Power"
- board text removed: "USB Hub"

Commit message: Add run_kicad_purge 4
Routing:
- net Net-(J101-D+): track 5.25 -> 4.56 mm
- net +5VPROTECTED: track 205.7 -> 205.0 mm
- net +3V3: track 99.4 -> 98.8 mm
