File: kicad/octohub4_v0.1/pcb_octohub4.kicad_pcb (KiCad board)
At the start: 2 copper layers, 100 x 80 mm, 83 parts, among them J101 USB231ARY, J102 USB231ARY, J103 USB231ARY, J104 USB231ARY, J201 Screw_Terminal_01x02, J203 Barrel_Jack_Switch, J301 USB_C_Receptacle_USB2.0, U201 TPS259474LRPWR, U301 AMS1117-3.3, U302 USB2514B_Bi, Y301 24MHz

Commit message: Add run_kicad_purge 5
Parts:
- R201: value 137 -> 120
Routing:
- net +5VPROTECTED: track 205.0 -> 203.7 mm
Changed lines of the file:
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@@
 		)
 		(fp_text user "${REFERENCE}"
-			(at 0 9 0)
+			(at 0 3 0)
 			(layer "F.Fab")
 			(effects
@@
 			)
 		)
-		(property "JLC" "C720524"
+		(property "JLC" "C720525"
 			(at 0 0 0)
 			(unlocked yes)
@@
 			)
 		)
-		(property "JLC" "C720524"
+		(property "JLC" "C720525"
 			(at 0 0 0)
 			(unlocked yes)
@@
 			)
 		)
-		(property "JLC" "C720524"
+		(property "JLC" "C720525"
 			(at 0 0 0)
 			(unlocked yes)
@@
 		(sheetname "/Power Protection/")
 		(sheetfile "pcb_octohub4_usbhubchip_power_protection.kicad_sch")
-		(attr through_hole)
+		(attr through_hole exclude_from_bom)
 		(fp_line
 			(start 8.92 -5.12)
@@
 			)
 		)
-		(property "Value" "137"
+		(property "Value" "120"
 			(at 0 1.65 0)
 			(layer "F.Fab")
@@
 			)
 		)
-		(property "JLC" "C720524"
+		(property "JLC" "C720525"
 			(at 0 0 0)
 			(unlocked yes)
@@
 	)
 	(gr_text "*"
-		(at 123.86 80.86 90)
+		(at 98.26 68.76 0)
 		(layer "F.SilkS")
 		(effects
@@
 	)
 	(gr_text "*"
-		(at 65.5726 61.91975 90)
+		(at 123.86 80.86 90)
 		(layer "F.SilkS")
 		(effects
@@
 		)
 	)
+	(gr_text "*"
+		(at 78.76 74.86 0)
+		(layer "F.SilkS")
+		(effects
+			(font
+				(size 1.5 1.5)
+				(thickness 0.3)
+				(bold yes)
+			)
+			(justify left bottom)
+		)
+	)
 	(gr_text "+5V\nUPSTREAM"
 		(at 83.97 71.9 0)
@@
 		)
 	)
-	(gr_text "*"
-		(at 39.7862 88.0752 90)
-		(layer "F.SilkS")
-		(effects
-			(font
-				(size 1.5 1.5)
-				(thickness 0.3)
-				(bold yes)
-			)
-			(justify left bottom)
-		)
-	)
 	(gr_text "5V IN"
 		(at 143.16 21.47 0)
@@
 		)
 	)
+	(gr_text "GND"
+		(at 61.76 96.26 0)
+		(layer "F.SilkS")
+		(effects
+			(font
+				(size 1 1)
+				(thickness 0.1875)
+			)
+			(justify left bottom)
+		)
+	)
 	(gr_text "${TITLE}\n${ISSUE_DATE} v${REVISION}"
 		(locked yes)
@@
 		)
 	)
+	(gr_text "*"
+		(at 131.05 75.56 90)
+		(layer "F.SilkS")
+		(effects
+			(font
+				(size 1.5 1.5)
+				(thickness 0.3)
+				(bold yes)
+			)
+			(justify left bottom)
+		)
+	)
 	(gr_text "+5V IN"
 		(at 86.76 26.76 0)
@@
 		)
 	)
+	(gr_text "*"
+		(at 121.26 65.96 0)
+		(layer "F.SilkS")
+		(effects
+			(font
+				(size 1.5 1.5)
+				(thickness 0.3)
+				(bold yes)
+			)
+			(justify left bottom)
+		)
+	)
+	(gr_text "*"
+		(at 78.76 71.26 0)
+		(layer "F.SilkS")
+		(effects
+			(font
+				(size 1.5 1.5)
+				(thickness 0.3)
+				(bold yes)
+			)
+			(justify left bottom)
+		)
+	)
+	(gr_text "GND"
+		(at 153.76 96.26 0)
+		(layer "F.SilkS")
+		(effects
+			(font
+				(size 1 1)
+				(thickness 0.1875)
+			)
+			(justify left bottom)
+		)
+	)
 	(gr_text "5V power distribution"
 		(at 102.56 20.56 0)
@@
 		)
 	)
+	(gr_text "*"
+		(at 73.76 64.66 0)
+		(layer "F.SilkS")
+		(effects
+			(font
+				(size 1.5 1.5)
+				(thickness 0.3)
+				(bold yes)
+			)
+			(justify left bottom)
+		)
+	)
 	(gr_text "5V IN\nBarrel Jack"
 		(at 98.205 29.376782 0)
@@
 		)
 	)
-	(gr_text_box "eFuse\n4A"
+	(gr_text_box "eFuse\n5.1A"
 		(start 109.305 22.813218)
 		(end 118.415 29.106782)
@@
 	)
 	(segment
-		(start 135.26 90.36)
-		(end 137.16 92.26)
-		(width 2)
-		(layer "F.Cu")
-		(net 2)
-	)
-	(segment
-		(start 115.593333 84.05)
-		(end 115.593333 90.493333)
-		(width 2)
-		(layer "F.Cu")
-		(net 2)
-	)
-	(segment
 		(start 78.191 80.806)
 		(end 78.191 81.46)
@@
 	)
 	(segment
-		(start 95.926667 90.426667)
-		(end 95.926667 84.05)
-		(width 2)
-		(layer "F.Cu")
-		(net 2)
-	)
-	(segment
-		(start 136.06 91.96)
-		(end 135.76 92.26)
-		(width 0.2)
-		(layer "F.Cu")
-		(net 2)
-	)
-	(segment
 		(start 76.26 90.26)
 		(end 78.26 92.26)
@@
 	)
 	(segment
-		(start 96.76 92.26)
-		(end 96.76 91.26)
-		(width 0.2)
-		(layer "F.Cu")
-		(net 2)
-	)
-	(segment
-		(start 116.66 92.26)
-		(end 135.76 92.26)
+		(start 115.593333 84.05)
+		(end 115.593333 92.226667)
 		(width 2)
 		(layer "F.Cu")
@@
 	)
 	(segment
-		(start 96.76 92.26)
-		(end 116.66 92.26)
-		(width 2)
-		(layer "F.Cu")
-		(net 2)
-	)
-	(segment
 		(start 120.711 82.06)
 		(end 119.06 82.06)
@@
 	)
 	(segment
-		(start 115.593333 90.493333)
-		(end 116.66 91.56)
-		(width 2)
-		(layer "F.Cu")
-		(net 2)
-	)
-	(segment
 		(start 81.56 77.76)
 		(end 78.26 77.76)
@@
 	(segment
 		(start 78.26 92.26)
-		(end 96.76 92.26)
+		(end 135.76 92.26)
 		(width 2)
 		(layer "F.Cu")
@@
 	)
 	(segment
-		(start 135.26 84.05)
-		(end 135.26 90.36)
+		(start 135.26 91.76)
+		(end 135.76 92.26)
+		(width 2)
+		(layer "F.Cu")
+		(net 2)
+	)
+	(segment
+		(start 95.926667 92.093333)
+		(end 95.926667 84.05)
 		(width 2)
 		(layer "F.Cu")
@@
 	)
 	(segment
-		(start 76.26 84.05)
-		(end 76.26 90.26)
+		(start 135.26 84.05)
+		(end 135.26 91.76)
 		(width 2)
 		(layer "F.Cu")
@@
 	)
 	(segment
-		(start 96.76 91.26)
-		(end 95.926667 90.426667)
+		(start 76.26 84.05)
+		(end 76.26 90.26)
 		(width 2)
 		(layer "F.Cu")
