File: kicad/octohub4_v0.1/pcb_octohub4_usbhubchip.kicad_sch (KiCad schematic)
At the start: 34 parts, among them J301 USB_C_Receptacle_USB2.0, U302 USB2514B_Bi, Y301 24MHz

Commit message: tmp
Parts:
- added BP204: Scope 5V OUT, 00_project_library:octoprobe_breakout_PB, symbol 00_project_library:octoprobe_breakout_BP
- added BP205: Scope 5V IN, 00_project_library:octoprobe_breakout_PB, symbol 00_project_library:octoprobe_breakout_BP
- added C311, C312: 10u, Capacitor_SMD:C_0603_1608Metric, symbol 00_project_library:C
- added U301: AMS1117-3.3, 00_project_library:SOT-223-3_TabPin2, symbol 00_project_library:AMS1117-3.3
Connections:
- net +3V3: now also C312.1, U301.2 (VO)
- net GND: now also C311.2, C312.2, U301.1 (GND)
- net HUB+5V renamed +5VIN
- net +5VIN: now also BP205.1; no longer R301.2, R305.2
- new net +5VOUT: BP204.1, C311.1, R301.2, R305.2, U301.3 (VI)
Other:
- note added: "Main Regulator Hub"
- note added: "Scope Pads"
- note removed: "Scope GND Pad"
- moved on the sheet: BP203, C301, C302, C303, C304, C307, C308, D301, R301, Y301

Commit message: Add run_kicad_purge 2
Parts:
- added D201, D202: SS34, Diode_SMD:D_SMA, symbol Diode:SS34
- added JP203: SolderJumper_2_Open, Jumper:SolderJumper-2_P1.3mm_Open_RoundedPad1.0x1.5mm, symbol Jumper:SolderJumper_2_Open
- added JP204: SolderJumper_2_Bridged, Jumper:SolderJumper-2_P1.3mm_Bridged_RoundedPad1.0x1.5mm, symbol Jumper:SolderJumper_2_Bridged
Connections:
- net +5VIN: no longer C401.2, D302.5 (VCC), J301.A4 (VBUS), J301.A9 (VBUS), J301.B4 (VBUS), J301.B9 (VBUS)
- removed net +5VOUT: BP204.1, C311.1, R301.2, R305.2, U301.3 (VI)
- new net: C311.1, D201.1 (K), D202.1 (K), U301.3 (VI)
- new net: D202.2 (A), JP204.1 (A)
- new net: D201.2 (A), JP203.1 (A)
- new net +5VPROTECTED: BP204.1, JP203.2 (B)
- new net +5VUPSTREAM: C401.2, D302.5 (VCC), J301.A4 (VBUS), J301.A9 (VBUS), J301.B4 (VBUS), J301.B9 (VBUS), JP204.2 (B), R301.2, R305.2
Other:
- moved on the sheet: C305, C311, C312, R304, U301

Commit message: Add run_kicad_purge 3
Parts:
- D301: Label LED_PWR (green) -> UPSTREAM_PWR (green)
Other:
- note added: "UPSTREAM POWER (USBC)"
- note removed: "Power LED"
- moved on the sheet: C305, C306, R304, R305, R306

Commit message: New via constraints: Copy usb hub footprint from tentacle v0.7
Parts:
- U302: footprint Package_DFN_QFN:Texas_RHH0036C_VQFN-36-1EP_6x6mm_P0.5mm_EP4.4x4.4mm_ThermalVias -> 00_project_library:Texas_RHH0036C_VQFN-36-1EP_6x6mm_P0.5mm_EP4.4x4.4mm_ThermalVias
Changed lines of the file:
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@@
 			)
 		)
-		(property "Footprint" "Package_DFN_QFN:Texas_RHH0036C_VQFN-36-1EP_6x6mm_P0.5mm_EP4.4x4.4mm_ThermalVias"
+		(property "Footprint" "00_project_library:Texas_RHH0036C_VQFN-36-1EP_6x6mm_P0.5mm_EP4.4x4.4mm_ThermalVias"
 			(at 245.11 114.3 0)
 			(effects
