File: kicad/octohub4_v0.2/pcb_octohub4_usbhubchip_power_protection.kicad_sch (KiCad schematic)
At the start: 25 parts, among them J201 Screw_Terminal_01x02, J203 Barrel_Jack_Switch, U201 TPS259474LRPWR

Commit message: v0.2: Update schematics and layout
Parts:
- added R204: 47k, Resistor_SMD:R_0805_2012Metric, symbol Device:R
- added R205: 24k, Resistor_SMD:R_0805_2012Metric, symbol Device:R
- added R206: 150k, Resistor_SMD:R_0805_2012Metric, symbol Device:R
- added R207: 220k, Resistor_SMD:R_0805_2012Metric, symbol Device:R
- added R208: 100k, Resistor_SMD:R_0805_2012Metric, symbol Device:R
Connections:
- net +5VIN: now also JP205.1 (A), R203.2, R204.2; no longer JP205.2 (B), U201.1 (EN_UVLO)
- net +5VPROTECTED: now also JP205.2 (B), R207.2; no longer JP205.1 (A), R203.2
- net GND: now also R206.1, R208.1; no longer U201.2 (OVCSEL)
- net at U201.3 (PG): now also D208.1 (K)
- net at U201.4 (PGTH): now also R207.1, R208.2; no longer D208.1 (K)
- new net: R204.1, R205.2, U201.1 (EN_UVLO)
- new net: R205.1, R206.2, U201.2 (OVLO)
- no-connect marks 1 -> 0
Other:
- moved on the sheet: D208, JP205, R203

Commit message: Recalculate all resistors around TPS25047
Parts:
- R201: JLCPCB (none) -> C17798
- R204: value 47k -> 330k; JLCPCB C17713 -> C23137
- R205: value 24k -> 18k; JLCPCB C17575 -> C25810
- R206: value 150k -> 100k; JLCPCB C17470 -> C149504
- R207: value 220k -> 120k; JLCPCB C17556 -> C25808
- R208: value 100k -> 47k; JLCPCB C25611 -> C17713
Changed lines of the file:
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@@
 			)
 		)
-		(property "Value" "100k"
+		(property "Value" "47k"
 			(at 147.2184 97.79 90)
 			(effects
@@
 			)
 		)
-		(property "JLCPCB" "C25611"
+		(property "JLCPCB" "C17713"
 			(at 147.32 97.79 90)
 			(effects
@@
 			)
 		)
-		(property "Value" "47k"
+		(property "Value" "330k"
 			(at 71.0184 91.44 90)
 			(effects
@@
 			)
 		)
-		(property "JLCPCB" "C17713"
+		(property "JLCPCB" "C23137"
 			(at 71.12 91.44 90)
 			(effects
@@
 			)
 		)
-		(property "Value" "24k"
+		(property "Value" "18k"
 			(at 71.0184 102.87 90)
 			(effects
@@
 			)
 		)
-		(property "JLCPCB" "C17575"
+		(property "JLCPCB" "C25810"
 			(at 71.12 102.87 90)
 			(effects
@@
 			)
 		)
-		(property "Value" "150k"
+		(property "Value" "100k"
 			(at 71.0184 118.11 90)
 			(effects
@@
 			)
 		)
-		(property "JLCPCB" "C17470"
+		(property "JLCPCB" "C149504"
 			(at 71.12 118.11 90)
 			(effects
@@
 			)
 		)
+		(property "JLCPCB" "C17798"
+			(at 146.05 125.73 90)
+			(effects
+				(font
+					(size 1.27 1.27)
+				)
+				(hide yes)
+			)
+		)
 		(pin "1"
 		)
@@
 			)
 		)
-		(property "Value" "220k"
+		(property "Value" "120k"
 			(at 147.2184 90.17 90)
 			(effects
@@
 			)
 		)
-		(property "JLCPCB" "C17556"
+		(property "JLCPCB" "C25808"
 			(at 147.32 90.17 90)
 			(effects
